File: pcb/FOX-JACK_EXT_BOARD_TOP/FOX-JACK_EXT_BOARD_TOP.kicad_sch (KiCad schematic)
At the start: 29 parts, among them J1 PICO_PIN_1-20, J4 PICO_PIN_21-40, Q1 FS8205, Q2 AO3401A, U1 TP4056-42-ESOP8, U2 DW01A

Commit message: UPDATE PCB
Parts:
- PS1: value ME2108A33P -> ME2108A50PG
Changed lines of the file:
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@@
 			)
 		)
-		(property "Value" "ME2108A33P"
+		(property "Value" "ME2108A50PG"
 			(at 234.95 68.58 0)
 			(effects
